File: hub-proto02/hub-proto02.brd (EAGLE design)
At the start: 87.3 x 26.7 mm, 10 parts

Commit message: refinements
Parts:
- renumbered STUB1 to SPUR1, STUB2 to SPUR2, STUB3 to SPUR3, STUB4 to SPUR4
Changed lines of the file:
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@@
 <attribute name="MF" value="" x="81.28" y="12.7" size="1.778" layer="27" rot="R270" display="off"/>
 </element>
-<element name="STUB1" library="con-amp-quick" package="06P" value="" x="68.58" y="12.7" rot="R270">
+<element name="SPUR1" library="con-amp-quick" package="06P" value="" x="68.58" y="12.7" rot="R270">
 <attribute name="OC_FARNELL" value="unknown" x="68.58" y="12.7" size="1.778" layer="27" rot="R270" display="off"/>
 <attribute name="MPN" value="" x="68.58" y="12.7" size="1.778" layer="27" rot="R270" display="off"/>
@@
 <attribute name="MF" value="" x="68.58" y="12.7" size="1.778" layer="27" rot="R270" display="off"/>
 </element>
-<element name="STUB2" library="con-amp-quick" package="06P" value="" x="54.61" y="12.7" rot="R270">
+<element name="SPUR2" library="con-amp-quick" package="06P" value="" x="54.61" y="12.7" rot="R270">
 <attribute name="OC_FARNELL" value="unknown" x="54.61" y="12.7" size="1.778" layer="27" rot="R270" display="off"/>
 <attribute name="MPN" value="" x="54.61" y="12.7" size="1.778" layer="27" rot="R270" display="off"/>
@@
 <attribute name="MF" value="" x="54.61" y="12.7" size="1.778" layer="27" rot="R270" display="off"/>
 </element>
-<element name="STUB3" library="con-amp-quick" package="06P" value="" x="40.64" y="12.7" rot="R270">
+<element name="SPUR3" library="con-amp-quick" package="06P" value="" x="40.64" y="12.7" rot="R270">
 <attribute name="OC_FARNELL" value="unknown" x="40.64" y="12.7" size="1.778" layer="27" rot="R270" display="off"/>
 <attribute name="MPN" value="" x="40.64" y="12.7" size="1.778" layer="27" rot="R270" display="off"/>
@@
 <attribute name="MF" value="" x="40.64" y="12.7" size="1.778" layer="27" rot="R270" display="off"/>
 </element>
-<element name="STUB4" library="con-amp-quick" package="06P" value="" x="25.4" y="12.7" rot="R270">
+<element name="SPUR4" library="con-amp-quick" package="06P" value="" x="25.4" y="12.7" rot="R270">
 <attribute name="OC_FARNELL" value="unknown" x="25.4" y="12.7" size="1.778" layer="27" rot="R270" display="off"/>
 <attribute name="MPN" value="" x="25.4" y="12.7" size="1.778" layer="27" rot="R270" display="off"/>
@@
 <signal name="+12V">
 <contactref element="CTRL" pad="1"/>
-<contactref element="STUB1" pad="1"/>
-<contactref element="STUB2" pad="1"/>
-<contactref element="STUB3" pad="1"/>
-<contactref element="STUB4" pad="1"/>
+<contactref element="SPUR1" pad="1"/>
+<contactref element="SPUR2" pad="1"/>
+<contactref element="SPUR3" pad="1"/>
+<contactref element="SPUR4" pad="1"/>
 <contactref element="TERM" pad="1"/>
 <wire x1="11.43" y1="19.05" x2="25.4" y2="19.05" width="1.016" layer="1"/>
@@
 <contactref element="CTRL" pad="6"/>
 <contactref element="TERM" pad="6"/>
-<contactref element="STUB1" pad="6"/>
-<contactref element="STUB2" pad="6"/>
-<contactref element="STUB3" pad="6"/>
-<contactref element="STUB4" pad="6"/>
+<contactref element="SPUR1" pad="6"/>
+<contactref element="SPUR2" pad="6"/>
+<contactref element="SPUR3" pad="6"/>
+<contactref element="SPUR4" pad="6"/>
 <polygon width="0.254" layer="1">
 <vertex x="0" y="26.67"/>
@@
 <signal name="CANH-IN">
 <contactref element="CTRL" pad="2"/>
-<contactref element="STUB1" pad="4"/>
+<contactref element="SPUR1" pad="4"/>
 <wire x1="68.58" y1="11.43" x2="71.12" y2="11.43" width="0.6096" layer="1"/>
 <wire x1="71.12" y1="11.43" x2="76.2" y2="16.51" width="0.6096" layer="1"/>
@@
 <signal name="CANL-IN">
 <contactref element="CTRL" pad="3"/>
-<contactref element="STUB1" pad="5"/>
+<contactref element="SPUR1" pad="5"/>
 <wire x1="68.58" y1="8.89" x2="72.39" y2="8.89" width="0.6096" layer="1"/>
 <wire x1="81.28" y1="13.97" x2="77.47" y2="13.97" width="0.6096" layer="1"/>
@@
 </signal>
 <signal name="N$5">
-<contactref element="STUB1" pad="2"/>
-<contactref element="STUB2" pad="4"/>
+<contactref element="SPUR1" pad="2"/>
+<contactref element="SPUR2" pad="4"/>
 <wire x1="54.61" y1="11.43" x2="57.15" y2="11.43" width="0.6096" layer="1"/>
 <wire x1="57.15" y1="11.43" x2="62.23" y2="16.51" width="0.6096" layer="1"/>
@@
 </signal>
 <signal name="N$6">
-<contactref element="STUB1" pad="3"/>
-<contactref element="STUB2" pad="5"/>
+<contactref element="SPUR1" pad="3"/>
+<contactref element="SPUR2" pad="5"/>
 <wire x1="54.61" y1="8.89" x2="58.42" y2="8.89" width="0.6096" layer="1"/>
 <wire x1="68.58" y1="13.97" x2="63.5" y2="13.97" width="0.6096" layer="1"/>
@@
 </signal>
 <signal name="N$7">
-<contactref element="STUB4" pad="2"/>
+<contactref element="SPUR4" pad="2"/>
 <contactref element="TERM" pad="4"/>
 <wire x1="11.43" y1="11.43" x2="13.97" y2="11.43" width="0.6096" layer="1"/>
@@
 </signal>
 <signal name="N$8">
-<contactref element="STUB4" pad="3"/>
+<contactref element="SPUR4" pad="3"/>
 <contactref element="TERM" pad="5"/>
 <wire x1="11.43" y1="8.89" x2="15.24" y2="8.89" width="0.6096" layer="1"/>
@@
 </signal>
 <signal name="N$9">
-<contactref element="STUB2" pad="3"/>
-<contactref element="STUB3" pad="5"/>
+<contactref element="SPUR2" pad="3"/>
+<contactref element="SPUR3" pad="5"/>
 <wire x1="40.64" y1="8.89" x2="44.45" y2="8.89" width="0.6096" layer="1"/>
 <wire x1="44.45" y1="8.89" x2="49.53" y2="13.97" width="0.6096" layer="1"/>
@@
 </signal>
 <signal name="N$10">
-<contactref element="STUB2" pad="2"/>
-<contactref element="STUB3" pad="4"/>
+<contactref element="SPUR2" pad="2"/>
+<contactref element="SPUR3" pad="4"/>
 <wire x1="40.64" y1="11.43" x2="43.18" y2="11.43" width="0.6096" layer="1"/>
 <wire x1="43.18" y1="11.43" x2="48.26" y2="16.51" width="0.6096" layer="1"/>
@@
 </signal>
 <signal name="N$11">
-<contactref element="STUB3" pad="3"/>
-<contactref element="STUB4" pad="5"/>
+<contactref element="SPUR3" pad="3"/>
+<contactref element="SPUR4" pad="5"/>
 <wire x1="25.4" y1="8.89" x2="29.21" y2="8.89" width="0.6096" layer="1"/>
 <wire x1="29.21" y1="8.89" x2="34.29" y2="13.97" width="0.6096" layer="1"/>
@@
 </signal>
 <signal name="N$12">
-<contactref element="STUB3" pad="2"/>
-<contactref element="STUB4" pad="4"/>
+<contactref element="SPUR3" pad="2"/>
+<contactref element="SPUR4" pad="4"/>
 <wire x1="25.4" y1="11.43" x2="27.94" y2="11.43" width="0.6096" layer="1"/>
 <wire x1="27.94" y1="11.43" x2="33.02" y2="16.51" width="0.6096" layer="1"/>
@@
 <signal name="CANL-OUT">
 <contactref element="TERM" pad="3"/>
-<contactref element="TERM_R" pad="1"/>
 <wire x1="11.43" y1="13.97" x2="10.16" y2="13.97" width="0.6096" layer="16"/>
 <wire x1="10.16" y1="13.97" x2="8.89" y2="12.7" width="0.6096" layer="16"/>
-<wire x1="5.08" y1="3.81" x2="7.62" y2="3.81" width="0.6096" layer="16"/>
 <wire x1="7.62" y1="3.81" x2="8.89" y2="5.08" width="0.6096" layer="16"/>
 <wire x1="8.89" y1="5.08" x2="8.89" y2="12.7" width="0.6096" layer="16"/>
+<contactref element="TERM_R" pad="1"/>
+<wire x1="7.62" y1="3.81" x2="5.08" y2="3.81" width="0.6096" layer="16"/>
 </signal>
 <signal name="CANH-OUT">
